File: fan_controller.sch (KiCad schematic (older format))
At the start: 86 parts, among them J1 SM04B-SRSS-TB, J10 DNI_47053-1000, J11 DNI_26-01-3114, J2 SM04B-SRSS-TB, J3 SM04B-SRSS-TB, J4 SM04B-SRSS-TB, J5 DNI_53047-0310, J6 DNI_53047-0310, J7 DNI_47053-1000, J8 DNI_26-01-3115, J9 DNI_47053-1000, U1 PCA9546APW, U2 INA3221, U3 W25Q64JVSSIM, U4 OPA2313QDGKRQ1, U5 SN74AHCT125PW

Commit message: rev2: swap D31 and D32 at U3
Connections:
- net D31: now also R20.2, U3.1 (~CS); no longer U3.6 (CLK)
- net D32: now also U3.6 (CLK); no longer R20.2, U3.1 (~CS)
Changed lines of the file:
@@
 Title "fan controller"
 Date "2021-10-31"
-Rev "1"
+Rev "2"
 Comp "alexth4ef9"
 Comment1 "Copyright alexth4f9 2021"
@@
 	4950 9300 4950 9350
 Wire Wire Line
-	4450 8800 4350 8800
-Wire Wire Line
-	4350 8750 4350 8800
-Connection ~ 4350 8800
-Wire Wire Line
-	4350 8800 4100 8800
-Wire Wire Line
-	4450 9000 4100 9000
-Wire Wire Line
 	5450 9000 5900 9000
 Wire Wire Line
@@
 Text Label 5650 8800 0    50   ~ 0
 D33
+Text Label 4100 9000 0    50   ~ 0
+D32
 Text Label 4100 8800 0    50   ~ 0
-D32
-Text Label 4100 9000 0    50   ~ 0
 D31
 Wire Wire Line
@@
 Text Notes 12600 850  0    50   ~ 0
 OLIMEXINO-STM32F3 modification: wire between VIN and PWR1 pin 2
+Wire Wire Line
+	4450 9000 4100 9000
+Wire Wire Line
+	4450 8800 4350 8800
+Wire Wire Line
+	4350 8750 4350 8800
+Connection ~ 4350 8800
+Wire Wire Line
+	4350 8800 4100 8800
 $EndSCHEMATC

Commit message: rev3: fix stemma qt pinout
Connections:
- net +3V3: now also J1.2 (Pin_2), J2.2 (Pin_2), J4.2 (Pin_2); no longer J1.1 (Pin_1), J2.1 (Pin_1), J4.1 (Pin_1)
- net GND: now also J1.1 (Pin_1), J2.1 (Pin_1), J4.1 (Pin_1); no longer J1.2 (Pin_2), J2.2 (Pin_2), J4.2 (Pin_2)
