File: fan_controller.kicad_pcb (KiCad board)
At the start: 4 copper layers, 68.5 x 53.3 mm, 87 parts, among them J1 SM04B-SRSS-TB, J10 DNI_47053-1000, J11 DNI_26-01-3114, J2 SM04B-SRSS-TB, J3 SM04B-SRSS-TB, J4 SM04B-SRSS-TB, J5 DNI_53047-0310, J6 DNI_53047-0310, J7 DNI_47053-1000, J8 DNI_26-01-3115, J9 DNI_47053-1000, U1 PCA9546APW, U2 INA3221, U3 W25Q64JVSSIM, U4 OPA2313QDGKRQ1, U5 SN74AHCT125PW

Commit message: rev2: swap D31 and D32 at U3
Connections:
- R20 pad 2: /D32 -> /D31
- U3 pad 1: /D32 -> /D31
- U3 pad 6: /D31 -> /D32
Routing:
- net /D32: track 7.78 -> 13.6 mm, vias 0 -> 1
- net /D31: track 16.1 -> 11.4 mm, vias 1 -> 0
Other:
- board text added: "fan controller rev2"
Changed lines of the file:
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@@
     (thickness 1.6)
     (drawings 3)
-    (tracks 787)
+    (tracks 788)
     (zones 0)
     (modules 87)
@@
     (title "fan controller")
     (date 2021-10-31)
-    (rev 1)
+    (rev 2)
     (company alexth4ef9)
     (comment 1 "Copyright alexth4ef9 2021")
@@
     (add_net "Net-(U5-Pad11)")
   )
-  (module Symbol:OSHW-Logo2_9.8x8mm_SilkScreen (layer B.Cu)
+  (module Symbol:OSHW-Logo2_9.8x8mm_SilkScreen locked (layer B.Cu)
     (at 133.8 102.8 180)
     (descr "Open Source Hardware Symbol")
@@
       (net 74 "Net-(R28-Pad2)"))
     (pad 6 smd roundrect (at 3.6 0.635 270) (size 1.6 0.6) (layers F.Cu F.Paste F.Mask) (roundrect_rratio 0.25)
-      (net 34 /D31))
+      (net 35 /D32))
     (pad 5 smd roundrect (at 3.6 1.905 270) (size 1.6 0.6) (layers F.Cu F.Paste F.Mask) (roundrect_rratio 0.25)
       (net 26 /D34))
@@
       (net 27 /D33))
     (pad 1 smd roundrect (at -3.6 -1.905 270) (size 1.6 0.6) (layers F.Cu F.Paste F.Mask) (roundrect_rratio 0.25)
-      (net 35 /D32))
+      (net 34 /D31))
     (model ${KISYS3DMOD}/Package_SO.3dshapes/SOIC-8_5.23x5.23mm_P1.27mm.wrl
       (at (xyz 0 0 0))
@@
     )
     (pad 2 smd roundrect (at 0.825 0 90) (size 0.8 0.95) (layers F.Cu F.Paste F.Mask) (roundrect_rratio 0.25)
-      (net 35 /D32))
+      (net 34 /D31))
     (pad 1 smd roundrect (at -0.825 0 90) (size 0.8 0.95) (layers F.Cu F.Paste F.Mask) (roundrect_rratio 0.25)
       (net 9 +3V3))
@@
     )
   )
-  (gr_text "fan controller\nrev1" (at 132.6 118) (layer F.SilkS)
+  (gr_text "fan controller\nrev2" (at 132.6 118) (layer F.SilkS)
     (effects (font (size 1 1) (thickness 0.15)) (justify left))
   )
@@
   (segment (start 135.7 99.3) (end 136.95 98.05) (width 0.25) (layer F.Cu) (net 31))
   (segment (start 149 106.2) (end 149 102.6) (width 0.25) (layer F.Cu) (net 31))
-  (via (at 170.8 107.6) (size 0.8) (drill 0.4) (layers F.Cu B.Cu) (net 34))
-  (segment (start 169.565 108.835) (end 170.8 107.6) (width 0.25) (layer F.Cu) (net 34))
-  (segment (start 169.565 110.4) (end 169.565 108.835) (width 0.25) (layer F.Cu) (net 34))
-  (segment (start 173.473002 107.6) (end 170.8 107.6) (width 0.25) (layer B.Cu) (net 34))
-  (segment (start 177.973002 103.1) (end 173.473002 107.6) (width 0.25) (layer B.Cu) (net 34))
-  (segment (start 179.89118 103.1) (end 177.973002 103.1) (width 0.25) (layer B.Cu) (net 34))
-  (segment (start 181.16351 101.82767) (end 179.89118 103.1) (width 0.25) (layer B.Cu) (net 34))
-  (segment (start 172.105 103.2) (end 172.105 102.095) (width 0.25) (layer F.Cu) (net 35))
-  (segment (start 172.425 101.775) (end 175.2 101.775) (width 0.25) (layer F.Cu) (net 35))
-  (segment (start 172.105 102.095) (end 172.425 101.775) (width 0.25) (layer F.Cu) (net 35))
+  (segment (start 172.105 103.2) (end 172.105 102.095) (width 0.25) (layer F.Cu) (net 34))
+  (segment (start 172.425 101.775) (end 175.2 101.775) (width 0.25) (layer F.Cu) (net 34))
+  (segment (start 172.105 102.095) (end 172.425 101.775) (width 0.25) (layer F.Cu) (net 34))
+  (segment (start 177.5 103.1) (end 179.89118 103.1) (width 0.25) (layer F.Cu) (net 34))
+  (segment (start 179.89118 103.1) (end 181.16351 101.82767) (width 0.25) (layer F.Cu) (net 34))
+  (segment (start 176.175 101.775) (end 177.5 103.1) (width 0.25) (layer F.Cu) (net 34))
+  (segment (start 175.2 101.775) (end 176.175 101.775) (width 0.25) (layer F.Cu) (net 34))
+  (via (at 170.8 107.6) (size 0.8) (drill 0.4) (layers F.Cu B.Cu) (net 35))
+  (segment (start 169.565 108.835) (end 170.8 107.6) (width 0.25) (layer F.Cu) (net 35))
+  (segment (start 169.565 110.4) (end 169.565 108.835) (width 0.25) (layer F.Cu) (net 35))
   (segment (start 178.57084 101.775) (end 178.62351 101.82767) (width 0.25) (layer F.Cu) (net 35))
-  (segment (start 175.2 101.775) (end 178.57084 101.775) (width 0.25) (layer F.Cu) (net 35))
+  (segment (start 176.57233 101.82767) (end 178.62351 101.82767) (width 0.25) (layer B.Cu) (net 35))
+  (segment (start 170.8 107.6) (end 176.57233 101.82767) (width 0.25) (layer B.Cu) (net 35))
   (segment (start 171.8 78.3) (end 170.5 78.3) (width 0.25) (layer F.Cu) (net 36))
   (segment (start 169.2 77) (end 168.225 77) (width 0.25) (layer F.Cu) (net 36))

Commit message: rev3: fix stemma qt pinout
Connections:
- J1 pad 1: +3V3 -> GND
- J1 pad 2: GND -> +3V3
- J2 pad 1: +3V3 -> GND
- J2 pad 2: GND -> +3V3
- J4 pad 1: +3V3 -> GND
- J4 pad 2: GND -> +3V3
Other:
- board text added: "fan controller rev3"
- board text removed: "fan controller rev1"

Commit message: updated documentation
Other:
- board text removed: "fan controller rev2"
